File: hw/double_pt100/double_pt100.kicad_pcb (KiCad board)
At the start: 2 copper layers, 88.9 x 45.7 mm, 30 parts, among them SW1 SW_Push, U1 WeMos_D1_mini, U2 OLED_091_module, U3 MAX31865_breakout, U4 MAX31865_breakout

Commit message: hw version 0.2 with alternative assembly
Parts:
- added BZ1: Buzzer, Buzzer_Beeper:Buzzer_12x9.5RM7.6, F.Cu at (80.6, 129.6)
- added C10: 100n, Capacitor_SMD:C_0603_1608Metric, F.Cu at (107.3, 141.0)
- added C11: 100n, Capacitor_SMD:C_0603_1608Metric, F.Cu at (107.3, 136.5)
- added C12: 100n, Capacitor_SMD:C_0603_1608Metric, F.Cu at (107.3, 132.7)
- added C7: 100n, Capacitor_SMD:C_0603_1608Metric, F.Cu at (83.8, 106.7)
- added C8: 100n, Capacitor_SMD:C_0603_1608Metric, F.Cu at (83.8, 109.9)
- added C9: 100n, Capacitor_SMD:C_0603_1608Metric, F.Cu at (87.0, 138.4)
- added D1: LED, LED_SMD:LED_0805_2012Metric, F.Cu at (87.6, 128.3)
- added D2: BAV70, Package_TO_SOT_SMD:SOT-23, F.Cu at (100.3, 137.2)
- added D3: BAV70, Package_TO_SOT_SMD:SOT-23, F.Cu at (100.3, 131.4)
- added J1: Screw_Terminal_01x03, TerminalBlock:TerminalBlock_bornier-3_P5.08mm, F.Cu at (85.1, 144.8)
- added Q1: BC817, Package_TO_SOT_SMD:SOT-23, F.Cu at (90.2, 138.4)
- added R12: 330, Resistor_SMD:R_0603_1608Metric, F.Cu at (99.1, 141.0)
- added R13: 330, Resistor_SMD:R_0603_1608Metric, F.Cu at (104.8, 141.0)
- added R14: 10k, Resistor_SMD:R_0603_1608Metric, F.Cu at (95.2, 138.4)
- added R15: 10k, Resistor_SMD:R_0603_1608Metric, F.Cu at (90.2, 135.3)
- added R16: 1k0, Resistor_SMD:R_0603_1608Metric, F.Cu at (84.5, 125.1)
- added R17: 330, Resistor_SMD:R_0603_1608Metric, F.Cu at (101.0, 141.0)
- added R18: 330, Resistor_SMD:R_0603_1608Metric, F.Cu at (102.9, 141.0)
- added R19: 330, Resistor_SMD:R_0603_1608Metric, F.Cu at (81.3, 141.0)
- added R21: 330, Resistor_SMD:R_0603_1608Metric, F.Cu at (79.4, 141.0)
- added R22: 330, Resistor_SMD:R_0603_1608Metric, F.Cu at (77.5, 141.0)
- added R23: 10k, Resistor_SMD:R_0603_1608Metric, F.Cu at (93.3, 138.4)
- added Re: 330, Resistor_SMD:R_0603_1608Metric, F.Cu at (75.6, 141.0)
- added U5: RP2040-Zero-SideOnly, myModules:RP2040-Zero-SideOnly, F.Cu at (89.5, 115.6)
- added U6: LM7805_TO220, myModules:BUCK5V, F.Cu at (104.5, 134.6)
- moved R9 2.54 mm to (104.1, 130.2)
- moved R8 1.91 mm to (104.1, 128.3)
- moved R7 1.27 mm to (104.1, 126.4)
- moved C4 1.27 mm to (78.1, 125.7)
- moved R2 0.64 mm to (104.1, 124.5)
Connections:
- net Net-(R2-Pad1) renamed SWR
- net Net-(R3-Pad1) renamed SCLR
- net Net-(R4-Pad1) renamed SDAR
- net Net-(R5-Pad1) renamed CS1R
- net Net-(R6-Pad1) renamed CS2R
- net Net-(R7-Pad1) renamed CLKR
- net Net-(R8-Pad1) renamed SDOR
- net Net-(R9-Pad1) renamed SDIR
Routing:
- net GND: track 4.73 -> 97.0 mm, vias 31 -> 40
- net +5V: track 72.0 -> 128.7 mm, vias 1 -> 3
- net Net-(C9-Pad1): track 0.00 -> 20.1 mm
- net +3V3: track 95.0 -> 114.5 mm
- net Net-(C11-Pad1): track 0.00 -> 15.0 mm
- net Net-(C10-Pad1): track 0.00 -> 12.4 mm
- net Net-(C12-Pad1): track 0.00 -> 11.1 mm
- net Net-(D1-Pad1): track 0.00 -> 10.9 mm
- net Net-(J1-Pad3): track 0.00 -> 10.8 mm
- net Net-(J1-Pad1): track 0.00 -> 10.8 mm
- net SCLR: track 2.50 -> 11.6 mm
- net CS2R: track 2.51 -> 9.77 mm
- net CS1R: track 2.53 -> 9.13 mm
- net SDAR: track 2.50 -> 7.21 mm
- net BEEP: track 0.00 -> 4.35 mm
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Other:
- board text added: "OH 2303"
- board text added: "v0.2 2023.03"
- board text removed: "OH 2301"
- board text removed: "v0.1 2023.01"
