File: hw/double_pt100/double_pt100.kicad_pcb (KiCad board)
At the start: 2 copper layers, 88.9 x 45.7 mm, 28 parts, among them SW1 SW_Push, U1 WeMos_D1_mini, U2 OLED_091_module, U3 MAX31865_breakout, U4 MAX31865_breakout

Commit message: layout done
Routing:
- net +3V3: track 24.4 -> 95.0 mm
- net +5V: track 11.6 -> 72.7 mm, vias 0 -> 1
- net GND: track 0.70 -> 5.43 mm, vias 0 -> 31
- net CS2: track 13.6 -> 16.0 mm
- net SDA: track 25.0 -> 23.8 mm
- net CS1: track 49.0 -> 48.2 mm
- added copper zone on B.Cu, net GND
- added copper zone on F.Cu, net GND
Other:
- board text added: "OH 2301"
- board text added: "PT100 WiFi"
- board text added: "v0.1 2023.01"

Commit message: gerbers to order the prototype
Parts:
- added H7: MountingHole, MountingHole:MountingHole_3.2mm_M3, F.Cu at (147.3, 108.0)
- added H8: MountingHole, MountingHole:MountingHole_3.2mm_M3, F.Cu at (88.9, 108.0)
Routing:
- net +5V: track 72.7 -> 72.0 mm
- net GND: track 5.43 -> 4.73 mm
Changed lines of the file:
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@@
     (pad_to_mask_clearance 0)
     (pcbplotparams
-      (layerselection 0x00010fc_ffffffff)
+      (layerselection 0x00010e0_ffffffff)
       (disableapertmacros false)
       (usegerberextensions false)
@@
       (excludeedgelayer true)
       (plotframeref false)
-      (viasonmask false)
+      (viasonmask true)
       (mode 1)
       (useauxorigin false)
@@
       (outputformat 1)
       (mirror false)
-      (drillshape 1)
+      (drillshape 0)
       (scaleselection 1)
       (outputdirectory "")
@@
     )
   )
+  (footprint "MountingHole:MountingHole_3.2mm_M3" (layer "F.Cu")
+    (at 88.9 107.95)
+    (descr "Mounting Hole 3.2mm, no annular, M3")
+    (tags "mounting hole 3.2mm no annular m3")
+    (property "Sheetfile" "double_pt100.kicad_sch")
+    (property "Sheetname" "")
+    (attr exclude_from_pos_files)
+    (fp_text reference "H8" (at 0 -4.2) (layer "F.SilkS") hide
+      (effects (font (size 1 1) (thickness 0.15)))
+    )
+    (fp_text value "MountingHole" (at 0 4.2) (layer "F.Fab") hide
+      (effects (font (size 1 1) (thickness 0.15)))
+    )
+    (fp_text user "${REFERENCE}" (at 0 0) (layer "F.Fab") hide
+      (effects (font (size 1 1) (thickness 0.15)))
+    )
+    (fp_circle (center 0 0) (end 3.2 0) (layer "Cmts.User") (width 0.15) (fill none))
+    (fp_circle (center 0 0) (end 3.45 0) (layer "F.CrtYd") (width 0.05) (fill none))
+    (pad "" np_thru_hole circle (at 0 0) (size 3.2 3.2) (drill 3.2) (layers *.Cu *.Mask))
+  )
   (footprint "Resistor_SMD:R_0603_1608Metric" (layer "F.Cu")
     (at 104.14 118.0775)
@@
       (rotate (xyz 0 0 0))
     )
+  )
+  (footprint "MountingHole:MountingHole_3.2mm_M3" (layer "F.Cu")
+    (at 147.32 107.95)
+    (descr "Mounting Hole 3.2mm, no annular, M3")
+    (tags "mounting hole 3.2mm no annular m3")
+    (property "Sheetfile" "double_pt100.kicad_sch")
+    (property "Sheetname" "")
+    (attr exclude_from_pos_files)
+    (fp_text reference "H7" (at 0 -4.2) (layer "F.SilkS") hide
+      (effects (font (size 1 1) (thickness 0.15)))
+    )
+    (fp_text value "MountingHole" (at 0 4.2) (layer "F.Fab") hide
+      (effects (font (size 1 1) (thickness 0.15)))
+    )
+    (fp_text user "${REFERENCE}" (at 0 0) (layer "F.Fab") hide
+      (effects (font (size 1 1) (thickness 0.15)))
+    )
+    (fp_circle (center 0 0) (end 3.2 0) (layer "Cmts.User") (width 0.15) (fill none))
+    (fp_circle (center 0 0) (end 3.45 0) (layer "F.CrtYd") (width 0.05) (fill none))
+    (pad "" np_thru_hole circle (at 0 0) (size 3.2 3.2) (drill 3.2) (layers *.Cu *.Mask))
   )
   (footprint "Module:WEMOS_D1_mini_light" (layer "F.Cu")
@@
     (effects (font (size 1.2 1.2) (thickness 0.3)))
   )
-  (dimension (type aligned) (layer "Edge.Cuts")
+  (dimension (type aligned) (layer "Dwgs.User")
     (pts (xy 73.66 149.86) (xy 73.66 104.14))
     (height -10.16)
-    (gr_text "45,7200 mm" (at 62.35 127 90) (layer "Edge.Cuts")
+    (gr_text "45,7200 mm" (at 62.35 127 90) (layer "Dwgs.User")
       (effects (font (size 1 1) (thickness 0.15)))
     )
@@
     (style (thickness 0.1) (arrow_length 1.27) (text_position_mode 0) (extension_height 0.58642) (extension_offset 0.5) keep_text_aligned)
   )
-  (dimension (type aligned) (layer "Edge.Cuts")
+  (dimension (type aligned) (layer "Dwgs.User")
     (pts (xy 73.66 104.14) (xy 162.56 104.14))
     (height -10.16)
-    (gr_text "88,9000 mm" (at 118.11 92.83) (layer "Edge.Cuts")
+    (gr_text "88,9000 mm" (at 118.11 92.83) (layer "Dwgs.User")
       (effects (font (size 1 1) (thickness 0.15)))
     )
@@
   (segment (start 127.889 126.492) (end 129.921 124.46) (width 0.8) (layer "B.Cu") (net 1))
   (segment (start 156.21 123.19) (end 156.21 119.875) (width 0.8) (layer "F.Cu") (net 2))
-  (segment (start 101.31 122.695) (end 100.815 123.19) (width 0.4) (layer "F.Cu") (net 2))
   (segment (start 103.365 122.695) (end 102.87 123.19) (width 0.8) (layer "F.Cu") (net 2))
   (segment (start 156.21 119.875) (end 155.715 119.38) (width 0.8) (layer "F.Cu") (net 2))
@@
   (segment (start 119.57 107.95) (end 122.555 107.95) (width 0.4) (layer "F.Cu") (net 8))
   (via (at 107.061 109.855) (size 0.8) (drill 0.4) (layers "F.Cu" "B.Cu") (net 8))
-  (segment (start 119.634 109.982) (end 107.188 109.982) (width 0.4) (layer "B.Cu") (net 8))
-  (segment (start 122.555 108.204) (end 122.555 107.95) (width 0.4) (layer "B.Cu") (net 8))
+  (segment (start 120.523 109.982) (end 107.188 109.982) (width 0.4) (layer "B.Cu") (net 8))
   (segment (start 107.188 109.982) (end 107.061 109.855) (width 0.4) (layer "B.Cu") (net 8))
   (segment (start 122.555 107.95) (end 120.523 109.982) (width 0.4) (layer "B.Cu") (net 8))
-  (segment (start 120.523 109.982) (end 119.634 109.982) (width 0.4) (layer "B.Cu") (net 8))
   (segment (start 103.315 115.6475) (end 100.8925 115.6475) (width 0.4) (layer "F.Cu") (net 9))
   (segment (start 100.8925 115.6475) (end 100.815 115.57) (width 0.4) (layer "F.Cu") (net 9))
@@
   (segment (start 100.815 118.11) (end 103.2825 118.11) (width 0.4) (layer "F.Cu") (net 11))
   (segment (start 106.299 116.7435) (end 104.965 118.0775) (width 0.4) (layer "F.Cu") (net 12))
-  (segment (start 104.9975 118.11) (end 104.965 118.0775) (width 0.4) (layer "F.Cu") (net 12))
   (segment (start 106.299 116.713) (end 106.299 116.7435) (width 0.4) (layer "F.Cu") (net 12))
   (via (at 106.299 116.713) (size 0.8) (drill 0.4) (layers "F.Cu" "B.Cu") (net 12))
@@
   (segment (start 141.605 121.285) (end 143.51 123.19) (width 0.4) (layer "F.Cu") (net 18))
   (segment (start 108.585 122.555) (end 109.855 121.285) (width 0.4) (layer "F.Cu") (net 18))
-  (segment (start 101.31 121.145) (end 100.815 120.65) (width 0.4) (layer "F.Cu") (net 27))
   (segment (start 115.21 117.115) (end 115.57 117.475) (width 0.25) (layer "F.Cu") (net 27))
   (segment (start 108.585 114.44) (end 108.585 116.205) (width 0.25) (layer "F.Cu") (net 27))

Commit message: hw version mini
Parts:
- removed H1, H2, H3, H4, H5, H6, H7, H8: MountingHole, MountingHole:MountingHole_3.2mm_M3
- added J1: Screw_Terminal_01x02, TerminalBlock_Phoenix:TerminalBlock_Phoenix_PT-1,5-2-3.5-H_1x02_P3.50mm_Horizontal, F.Cu at (106.8, 125.0)
- moved C3 30.7 mm to (135.9, 127.6), turned to 0 degrees
- moved U4 30.5 mm to (88.3, 121.9)
- moved C2 30.2 mm to (97.2, 114.9)
- moved R1 30.0 mm to (80.6, 120.7), turned to 0 degrees
- moved R8 28.0 mm to (80.6, 114.9)
- moved R2 27.7 mm to (80.6, 110.5)
- moved R7 27.7 mm to (80.6, 113.0)
- moved R9 27.3 mm to (80.6, 118.7)
- moved SW1 25.1 mm to (135.9, 122.6)
- moved U3 20.7 mm to (126.4, 121.9)
- moved C6 20.1 mm to (135.3, 115.6)
- moved U2 17.8 mm to (104.8, 110.5)
- moved C5 12.8 mm to (106.7, 113.0)
- moved R10 11.5 mm to (107.3, 106.7), turned to 180 degrees
- moved R11 11.5 mm to (107.3, 109.2), turned to 180 degrees
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Routing:
- net SW: track 23.7 -> 80.7 mm, vias 0 -> 2
- net Net-(R7-Pad1): track 31.4 -> 1.86 mm
- net Net-(R2-Pad1): track 31.4 -> 1.86 mm
- net Net-(R8-Pad1): track 31.4 -> 2.13 mm
- net Net-(R9-Pad1): track 31.4 -> 2.13 mm
- net +3V3: track 95.0 -> 70.4 mm, vias 0 -> 1
- net CS1: track 48.2 -> 23.8 mm
- net SCL: track 21.0 -> 3.70 mm, vias 1 -> 0
- net +5V: track 72.0 -> 56.3 mm, vias 1 -> 0
- net SDA: track 23.5 -> 10.0 mm, vias 1 -> 0
- net CLK: track 55.5 -> 63.6 mm
- net SDO: track 54.0 -> 60.8 mm
- net SDI: track 52.5 -> 58.4 mm
- net GND: track 4.73 -> 1.58 mm, vias 31 -> 29
- net CS2: track 15.9 -> 13.9 mm
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Other:
- board size 88.9 x 45.7 mm -> 64.8 x 25.4 mm
- board text added: "+ -"
- board text added: "OH 2304"
- board text added: "v0.3 2023.04"
- board text removed: "OH 2301"
- board text removed: "v0.1 2023.01"
